File: ProjetArduino.brd (EAGLE design)
At the start: 44.1 x 69.8 mm, 55 parts, among them IC1 MEGA8-AI

Commit message: Version V1
Routing:
- net SCK: track 78.9 -> 133.8 mm
- net N$1: track 47.5 -> 79.0 mm
- net RESET: track 121.9 -> 90.9 mm
- net N$17: track 78.0 -> 51.6 mm, vias 0 -> 2
- net N$18: track 79.6 -> 53.6 mm
- net N$5: track 58.3 -> 39.1 mm
- net N$9: track 39.0 -> 57.9 mm, vias 2 -> 4
- net N$7: track 73.3 -> 57.5 mm
- net N$36: track 6.15 -> 19.8 mm, vias 1 -> 0
- net N$3: track 56.1 -> 68.9 mm
- net +5V: track 174.5 -> 161.9 mm
- net N$15: track 51.4 -> 40.3 mm
- net MOSI: track 90.0 -> 99.7 mm, vias 0 -> 2
- net N$19: track 64.5 -> 55.3 mm, vias 2 -> 4
- net N$21: track 78.2 -> 70.9 mm, vias 4 -> 3
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