File: eagle/v2.brd (EAGLE design)
At the start: 26.3 x 33 mm, 51 parts, among them IC1 MEGA8-AI

Commit message: Updae nano
Parts:
- RESET: device SparkFun:TACTILE_SWITCH_SMD -> lpatiny:TACTILE_SWITCH_SMD2
- moved JP1 22.2 mm to (24.8, 18.4)
- moved RESET 20.2 mm to (5.08, 18.4), flipped to the bottom, turned to 90 degrees
- moved RD5 9.16 mm to (10.2, 8.89)
- moved RC3 7.75 mm to (14.0, 27.9)
- moved R1 3.17 mm to (21.0, 14.0)
- moved RB5 2.84 mm to (21.0, 19.1), turned to 90 degrees
Routing:
- net RESET: track 38.7 -> 58.3 mm
- net N$20: track 24.1 -> 6.33 mm, vias 1 -> 0
- net N$13: track 27.0 -> 10.4 mm, vias 2 -> 0
- net N$4: track 21.7 -> 37.9 mm, vias 2 -> 0
- net N$8: track 43.7 -> 29.0 mm, vias 0 -> 2
- net N$21: track 21.7 -> 35.6 mm
- net N$17: track 13.2 -> 26.1 mm, vias 0 -> 2
- net N$36: track 2.49 -> 14.5 mm
- net N$15: track 15.0 -> 4.07 mm, vias 2 -> 0
- net N$1: track 21.1 -> 29.8 mm, vias 2 -> 4
- net N$46: track 9.04 -> 17.7 mm
- net N$14: track 20.8 -> 13.1 mm, vias 0 -> 2
- net N$28: track 2.29 -> 9.92 mm
- net GND: track 156.3 -> 162.8 mm
- net N$18: track 15.3 -> 9.70 mm, vias 2 -> 0
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