File: eagle/v2.sch (EAGLE design)
At the start: 51 parts, among them IC1 MEGA8-AI

Commit message: Updae nano
Parts:
- RESET: device SparkFun:TAC_SWITCHSMD -> lpatiny:TAC_SWITCH
Changed lines of the file:
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@@
 <part name="C1" library="eagle-ltspice" deviceset="C" device="C0603" value="0.1uF"/>
 <part name="C2" library="eagle-ltspice" deviceset="C" device="C0603" value="0.1uF"/>
-<part name="RESET" library="SparkFun" deviceset="TAC_SWITCH" device="SMD" value="Reset uC"/>
+<part name="RESET" library="lpatiny" deviceset="TAC_SWITCH" device="" value="Reset uC"/>
 </parts>
 <sheets>
