File: eagle/v3/v3.brd (EAGLE design)
At the start: 26.3 x 33 mm, 51 parts, among them IC1 MEGA8-AI

Commit message: Nouvelle version 0402 !!!!!!!!!!!!!
Parts:
- removed RESET: Reset uC, SparkFun:TACTILE_SWITCH_SMD
- added U$2: TEUCH4MM, florian:TEUCH4MM
- C1, C2: device eagle-ltspice:C0603 -> eagle-ltspice:C0402
- DB0, DB1, DB2, DB3, DB4, DB5, DB6, DB7, DC0, DC1, DC2, DC3, DC4, DC5, DD0, DD1, DD2, DD3, DD4, DD5, DD6, DD7: value (none) -> LED; device led:CHIPLED_0603 -> florian:D0402
- R1, RB0, RB1, RB2, RB3, RB4, RB5, RB6, RB7, RC0, RC1, RC2, RC3, RC4, RC5, RD0, RD1, RD2, RD3, RD4, RD5, RD6, RD7: device resistor:R0603 -> resistor:R0402
- moved JP1 22.2 mm to (24.8, 18.4)
- moved RD5 9.16 mm to (10.2, 8.89)
- moved RC3 7.75 mm to (14.0, 27.9)
- moved R1 3.17 mm to (21.0, 14.0)
- moved RB5 2.84 mm to (21.0, 19.1), turned to 90 degrees
Connections:
- new net N$22: U$2.1, U$2.4
- new net N$23: U$2.2, U$2.3
- net GND: no longer RESET.3
- net N$20: no longer RESET.1
Routing:
- net GND: track 156.3 -> 0.00 mm, vias 4 -> 0
- net +5V: track 77.1 -> 0.00 mm
- net N$8: track 43.7 -> 0.00 mm
- net SCK: track 43.7 -> 0.00 mm, vias 4 -> 0
- net RESET: track 38.7 -> 0.00 mm, vias 3 -> 0
- net MISO: track 34.5 -> 0.00 mm
- net N$13: track 27.0 -> 0.00 mm, vias 2 -> 0
- net MOSI: track 25.4 -> 0.00 mm, vias 3 -> 0
- net N$20: track 24.1 -> 0.00 mm, vias 1 -> 0
- net N$2: track 22.7 -> 0.00 mm, vias 2 -> 0
- net N$4: track 21.7 -> 0.00 mm, vias 2 -> 0
- net N$21: track 21.7 -> 0.00 mm
- net N$1: track 21.1 -> 0.00 mm, vias 2 -> 0
- net N$14: track 20.8 -> 0.00 mm
- net N$3: track 16.9 -> 0.00 mm
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
Commit message: Update smiley
Parts:
- removed DB4: LED, florian:D0402
- removed RB4: 1k, resistor:R0402
- added RD8: 10k, resistor:R0402
- added RD9: 1k, resistor:R0402
Connections:
- new net N$45: IC1.1, RD8.2
- net +5V: now also RD9.1
- net GND: now also RD8.1; no longer DB4.C
- net MISO: no longer IC1.16, RB4.1
- net MOSI: no longer IC1.15, RB3.1
- net N$11: now also IC1.17, RB5.1; no longer IC1.1, RD3.1
- net N$13: now also IC1.16, RB3.1; no longer IC1.9, RD5.1
- net N$14: now also IC1.15, RB2.1; no longer IC1.2, RD4.1
- net N$15: now also IC1.14, RB1.1; no longer IC1.10, RD6.1
- net N$16: now also IC1.13, RB0.1; no longer IC1.11, RD7.1
- net N$17: now also RD7.1; no longer RB0.1
- net N$18: now also IC1.11, RD6.1; no longer IC1.13, RB1.1
- net N$19: now also IC1.10, RD5.1; no longer IC1.14, RB2.1
- net N$20: now also IC1.9, RD4.1; no longer IC1.19
- net N$43: now also IC1.2, RD3.1; no longer DB4.A, RB4.2
- net SCK: no longer IC1.17, RB5.1

Commit message: Update library
Parts:
- removed JP1: (no value), SparkFun:SCREWTERMINAL-3.5MM-2
- added G1: CR2032H, florian:CR2032H
Connections:
- net +5V: now also G1.-; no longer JP1.1
- net GND: now also G1.+; no longer JP1.2
Changed lines of the file:
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@@
 <element name="CON1" library="lpatiny" package="TC2030-MCP-NL" value="" x="10.4775" y="4.445" rot="MR0"/>
 <element name="R1" library="resistor" package="R0402" value="10k" x="20.955" y="13.97" rot="MR270"/>
-<element name="JP1" library="SparkFun" package="SCREWTERMINAL-3.5MM-2" value="" x="24.765" y="18.415" rot="R90"/>
 <element name="C1" library="eagle-ltspice" package="C0402" value="0.1uF" x="15.875" y="31.75" rot="MR180">
 <attribute name="SPICEMODEL" value="NONE" x="15.875" y="31.75" size="1.778" layer="28" rot="MR180" display="off"/>
@@
 <element name="RD8" library="resistor" package="R0402" value="10k" x="1.905" y="-13.335"/>
 <element name="RD9" library="resistor" package="R0402" value="1k" x="1.905" y="-18.415"/>
+<element name="G1" library="florian" package="CR2032H" value="CR2032H" x="-10.16" y="-8.89"/>
 </elements>
 <signals>
@@
 <contactref element="DB6" pad="C"/>
 <contactref element="CON1" pad="GND"/>
-<contactref element="JP1" pad="2"/>
 <contactref element="IC1" pad="21"/>
 <contactref element="C2" pad="2"/>
@@
 <contactref element="DD5" pad="C"/>
 <contactref element="RD8" pad="1"/>
+<contactref element="G1" pad="+"/>
 <wire x1="20.97" y1="27.94" x2="20.97" y2="32.258" width="0" layer="19" extent="1-1"/>
 <wire x1="24.78" y1="27.94" x2="20.97" y2="27.94" width="0" layer="19" extent="1-1"/>
 <wire x1="17.16" y1="27.94" x2="20.97" y2="27.94" width="0" layer="19" extent="1-1"/>
 <wire x1="20.97" y1="23.495" x2="20.97" y2="27.94" width="0" layer="19" extent="1-1"/>
-<wire x1="24.765" y1="21.915" x2="20.97" y2="23.495" width="0" layer="19" extent="1-1"/>
 <wire x1="12.08" y1="27.94" x2="17.16" y2="27.94" width="0" layer="19" extent="1-1"/>
 <wire x1="8.27" y1="27.94" x2="12.08" y2="27.94" width="0" layer="19" extent="1-1"/>
@@
 <wire x1="26.05" y1="13.97" x2="20.97" y2="8.89" width="0" layer="19" extent="1-1"/>
 <wire x1="26.05" y1="3.81" x2="20.97" y2="8.89" width="0" layer="19" extent="1-1"/>
+<wire x1="-10.16" y1="1.27" x2="3.19" y2="3.81" width="0" layer="19" extent="1-1"/>
 <wire x1="1.255" y1="-13.335" x2="3.19" y2="3.81" width="0" layer="19" extent="1-1"/>
 </signal>
@@
 <contactref element="R1" pad="2"/>
 <contactref element="CON1" pad="5V"/>
-<contactref element="JP1" pad="1"/>
 <contactref element="IC1" pad="18"/>
 <contactref element="C2" pad="1"/>
 <contactref element="C1" pad="1"/>
 <contactref element="RD9" pad="1"/>
+<contactref element="G1" pad="-"/>
 <wire x1="12.08" y1="31.75" x2="15.225" y2="31.75" width="0" layer="19" extent="16-16"/>
 <wire x1="18.2626" y1="18.18" x2="15.225" y2="31.75" width="0" layer="19" extent="16-16"/>
 <wire x1="18.2626" y1="16.58" x2="18.2626" y2="18.18" width="0" layer="19" extent="16-16"/>
 <wire x1="20.955" y1="13.32" x2="18.2626" y2="16.58" width="0" layer="19" extent="16-16"/>
-<wire x1="24.765" y1="18.415" x2="20.955" y2="13.32" width="0" layer="19" extent="16-16"/>
 <wire x1="9.6774" y1="15.78" x2="18.2626" y2="16.58" width="0" layer="19" extent="16-16"/>
 <wire x1="9.2075" y1="5.08" x2="9.6774" y2="15.78" width="0" layer="19" extent="16-16"/>
 <wire x1="1.255" y1="-18.415" x2="9.2075" y2="5.08" width="0" layer="19" extent="1-16"/>
+<wire x1="-10.16" y1="-19.05" x2="1.255" y2="-18.415" width="0" layer="19" extent="1-1"/>
 </signal>
 <signal name="N$2">
