File: eagle/v3/v3.sch (EAGLE design)
At the start: 50 parts, among them IC1 MEGA8-AI

Commit message: Nouvelle version 0402 !!!!!!!!!!!!!
Parts:
- added U$2: TEUCH4MM, florian:TEUCH4MM
- C1, C2: device eagle-ltspice:CC0603 -> eagle-ltspice:CC0402
- DB0, DB1, DB2, DB3, DB4, DB5, DB6, DB7, DC0, DC1, DC2, DC3, DC4, DC5, DD0, DD1, DD2, DD3, DD4, DD5, DD6, DD7: value (none) -> LED; device led:LEDCHIPLED_0603 -> florian:LED
- R1, RB0, RB1, RB2, RB3, RB4, RB5, RB6, RB7, RC0, RC1, RC2, RC3, RC4, RC5, RD0, RD1, RD2, RD3, RD4, RD5, RD6, RD7: device resistor:R-EU_R0603 -> resistor:R-EU_R0402
Connections:
- new net N$20: IC1.ADC6
- new net N$22: U$2.1, U$2.2
- new net N$23: U$2.3, U$2.4
Changed lines of the file:
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@@
 <?xml version="1.0" encoding="utf-8"?>
 <!DOCTYPE eagle SYSTEM "eagle.dtd">
-<eagle version="6.5.0">
+<eagle version="7.2.0">
 <drawing>
 <settings>
@@
 <layer number="54" name="bGND_GNDA" color="1" fill="9" visible="no" active="no"/>
 <layer number="56" name="wert" color="7" fill="1" visible="no" active="no"/>
+<layer number="90" name="Modules" color="5" fill="1" visible="yes" active="yes"/>
 <layer number="91" name="Nets" color="2" fill="1" visible="yes" active="yes"/>
 <layer number="92" name="Busses" color="1" fill="1" visible="yes" active="yes"/>
@@
 <parts>
 <part name="IC1" library="atmel" deviceset="MEGA8" device="-AI"/>
-<part name="RC0" library="resistor" deviceset="R-EU_" device="R0603" value="1k"/>
-<part name="RC1" library="resistor" deviceset="R-EU_" device="R0603" value="1k"/>
-<part name="RC2" library="resistor" deviceset="R-EU_" device="R0603" value="1k"/>
-<part name="RC3" library="resistor" deviceset="R-EU_" device="R0603" value="1k"/>
-<part name="RC4" library="resistor" deviceset="R-EU_" device="R0603" value="1k"/>
-<part name="RC5" library="resistor" deviceset="R-EU_" device="R0603" value="1k"/>
-<part name="RD0" library="resistor" deviceset="R-EU_" device="R0603" value="1k"/>
-<part name="RD1" library="resistor" deviceset="R-EU_" device="R0603" value="1k"/>
-<part name="RD2" library="resistor" deviceset="R-EU_" device="R0603" value="1k"/>
-<part name="RD3" library="resistor" deviceset="R-EU_" device="R0603" value="1k"/>
-<part name="RD4" library="resistor" deviceset="R-EU_" device="R0603" value="1k"/>
-<part name="RD5" library="resistor" deviceset="R-EU_" device="R0603" value="1k"/>
-<part name="RD6" library="resistor" deviceset="R-EU_" device="R0603" value="1k"/>
-<part name="RD7" library="resistor" deviceset="R-EU_" device="R0603" value="1k"/>
-<part name="RB0" library="resistor" deviceset="R-EU_" device="R0603" value="1k"/>
-<part name="RB1" library="resistor" deviceset="R-EU_" device="R0603" value="1k"/>
-<part name="RB2" library="resistor" deviceset="R-EU_" device="R0603" value="1k"/>
-<part name="RB3" library="resistor" deviceset="R-EU_" device="R0603" value="1k"/>
-<part name="RB4" library="resistor" deviceset="R-EU_" device="R0603" value="1k"/>
-<part name="RB6" library="resistor" deviceset="R-EU_" device="R0603" value="1k"/>
-<part name="RB7" library="resistor" deviceset="R-EU_" device="R0603" value="1k"/>
-<part name="DB7" library="led" deviceset="LED" device="CHIPLED_0603"/>
-<part name="DC0" library="led" deviceset="LED" device="CHIPLED_0603"/>
-<part name="DC1" library="led" deviceset="LED" device="CHIPLED_0603"/>
-<part name="DC2" library="led" deviceset="LED" device="CHIPLED_0603"/>
-<part name="DC3" library="led" deviceset="LED" device="CHIPLED_0603"/>
-<part name="DC4" library="led" deviceset="LED" device="CHIPLED_0603"/>
-<part name="DC5" library="led" deviceset="LED" device="CHIPLED_0603"/>
-<part name="DD0" library="led" deviceset="LED" device="CHIPLED_0603"/>
-<part name="DD1" library="led" deviceset="LED" device="CHIPLED_0603"/>
-<part name="DD2" library="led" deviceset="LED" device="CHIPLED_0603"/>
-<part name="DD3" library="led" deviceset="LED" device="CHIPLED_0603"/>
-<part name="DD4" library="led" deviceset="LED" device="CHIPLED_0603"/>
-<part name="DD5" library="led" deviceset="LED" device="CHIPLED_0603"/>
-<part name="DD7" library="led" deviceset="LED" device="CHIPLED_0603"/>
-<part name="DB0" library="led" deviceset="LED" device="CHIPLED_0603"/>
-<part name="DB1" library="led" deviceset="LED" device="CHIPLED_0603"/>
-<part name="DB2" library="led" deviceset="LED" device="CHIPLED_0603"/>
-<part name="DB3" library="led" deviceset="LED" device="CHIPLED_0603"/>
-<part name="DB4" library="led" deviceset="LED" device="CHIPLED_0603"/>
-<part name="DB6" library="led" deviceset="LED" device="CHIPLED_0603"/>
-<part name="DD6" library="led" deviceset="LED" device="CHIPLED_0603"/>
+<part name="RC0" library="resistor" deviceset="R-EU_" device="R0402" value="1k"/>
+<part name="RC1" library="resistor" deviceset="R-EU_" device="R0402" value="1k"/>
+<part name="RC2" library="resistor" deviceset="R-EU_" device="R0402" value="1k"/>
+<part name="RC3" library="resistor" deviceset="R-EU_" device="R0402" value="1k"/>
+<part name="RC4" library="resistor" deviceset="R-EU_" device="R0402" value="1k"/>
+<part name="RC5" library="resistor" deviceset="R-EU_" device="R0402" value="1k"/>
+<part name="RD0" library="resistor" deviceset="R-EU_" device="R0402" value="1k"/>
+<part name="RD1" library="resistor" deviceset="R-EU_" device="R0402" value="1k"/>
+<part name="RD2" library="resistor" deviceset="R-EU_" device="R0402" value="1k"/>
+<part name="RD3" library="resistor" deviceset="R-EU_" device="R0402" value="1k"/>
+<part name="RD4" library="resistor" deviceset="R-EU_" device="R0402" value="1k"/>
+<part name="RD5" library="resistor" deviceset="R-EU_" device="R0402" value="1k"/>
+<part name="RD6" library="resistor" deviceset="R-EU_" device="R0402" value="1k"/>
+<part name="RD7" library="resistor" deviceset="R-EU_" device="R0402" value="1k"/>
+<part name="RB0" library="resistor" deviceset="R-EU_" device="R0402" value="1k"/>
+<part name="RB1" library="resistor" deviceset="R-EU_" device="R0402" value="1k"/>
+<part name="RB2" library="resistor" deviceset="R-EU_" device="R0402" value="1k"/>
+<part name="RB3" library="resistor" deviceset="R-EU_" device="R0402" value="1k"/>
+<part name="RB4" library="resistor" deviceset="R-EU_" device="R0402" value="1k"/>
+<part name="RB6" library="resistor" deviceset="R-EU_" device="R0402" value="1k"/>
+<part name="RB7" library="resistor" deviceset="R-EU_" device="R0402" value="1k"/>
+<part name="DB7" library="florian" deviceset="LED" device=""/>
+<part name="DC0" library="florian" deviceset="LED" device=""/>
+<part name="DC1" library="florian" deviceset="LED" device=""/>
+<part name="DC2" library="florian" deviceset="LED" device=""/>
+<part name="DC3" library="florian" deviceset="LED" device=""/>
+<part name="DC4" library="florian" deviceset="LED" device=""/>
+<part name="DC5" library="florian" deviceset="LED" device=""/>
+<part name="DD0" library="florian" deviceset="LED" device=""/>
+<part name="DD1" library="florian" deviceset="LED" device=""/>
+<part name="DD2" library="florian" deviceset="LED" device=""/>
+<part name="DD3" library="florian" deviceset="LED" device=""/>
+<part name="DD4" library="florian" deviceset="LED" device=""/>
+<part name="DD5" library="florian" deviceset="LED" device=""/>
+<part name="DD7" library="florian" deviceset="LED" device=""/>
+<part name="DB0" library="florian" deviceset="LED" device=""/>
+<part name="DB1" library="florian" deviceset="LED" device=""/>
+<part name="DB2" library="florian" deviceset="LED" device=""/>
+<part name="DB3" library="florian" deviceset="LED" device=""/>
+<part name="DB4" library="florian" deviceset="LED" device=""/>
+<part name="DB6" library="florian" deviceset="LED" device=""/>
+<part name="DD6" library="florian" deviceset="LED" device=""/>
 <part name="GND1" library="supply1" deviceset="GND" device=""/>
 <part name="P+3" library="supply1" deviceset="+5V" device=""/>
-<part name="RB5" library="resistor" deviceset="R-EU_" device="R0603" value="1k"/>
-<part name="DB5" library="led" deviceset="LED" device="CHIPLED_0603"/>
+<part name="RB5" library="resistor" deviceset="R-EU_" device="R0402" value="1k"/>
+<part name="DB5" library="florian" deviceset="LED" device=""/>
 <part name="GND2" library="supply1" deviceset="GND" device=""/>
 <part name="GND3" library="supply1" deviceset="GND" device=""/>
 <part name="CON1" library="lpatiny" deviceset="TINYISP" device="T"/>
-<part name="R1" library="resistor" deviceset="R-EU_" device="R0603" value="10k"/>
+<part name="R1" library="resistor" deviceset="R-EU_" device="R0402" value="10k"/>
 <part name="P+2" library="supply1" deviceset="+5V" device=""/>
 <part name="GND4" library="supply1" deviceset="GND" device=""/>
@@
 <part name="P+6" library="supply1" deviceset="+5V" device=""/>
 <part name="GND6" library="supply1" deviceset="GND" device=""/>
-<part name="C1" library="eagle-ltspice" deviceset="C" device="C0603" value="0.1uF"/>
-<part name="C2" library="eagle-ltspice" deviceset="C" device="C0603" value="0.1uF"/>
+<part name="C1" library="eagle-ltspice" deviceset="C" device="C0402" value="0.1uF"/>
+<part name="C2" library="eagle-ltspice" deviceset="C" device="C0402" value="0.1uF"/>
+<part name="U$2" library="florian" deviceset="TEUCH4MM" device=""/>
 </parts>
 <sheets>
@@
 <instance part="C1" gate="G$1" x="27.94" y="60.96" rot="R90"/>
 <instance part="C2" gate="G$1" x="7.62" y="33.02" rot="R180"/>
+<instance part="U$2" gate="G$1" x="128.524" y="53.594"/>
 </instances>
 <busses>
@@
 <junction x="114.3" y="55.88"/>
 <junction x="116.84" y="55.88"/>
+<wire x1="132.08" y1="58.42" x2="124.46" y2="58.42" width="0.1524" layer="91"/>
+<wire x1="124.46" y1="58.42" x2="116.84" y2="58.42" width="0.1524" layer="91"/>
+<wire x1="116.84" y1="58.42" x2="116.84" y2="55.88" width="0.1524" layer="91"/>
+<junction x="124.46" y="58.42"/>
+<junction x="132.08" y="58.42"/>
 </segment>
 <segment>
@@
 </segment>
 </net>
+<net name="N$20" class="0">
+<segment>
+<wire x1="132.08" y1="48.26" x2="124.46" y2="48.26" width="0.1524" layer="91"/>
+<wire x1="124.46" y1="48.26" x2="99.06" y2="48.26" width="0.1524" layer="91"/>
+<wire x1="99.06" y1="48.26" x2="99.06" y2="53.34" width="0.1524" layer="91"/>
+<pinref part="IC1" gate="G$1" pin="ADC6"/>
+<wire x1="99.06" y1="53.34" x2="83.82" y2="53.34" width="0.1524" layer="91"/>
+<junction x="83.82" y="53.34"/>
+<junction x="132.08" y="48.26"/>
+<junction x="124.46" y="48.26"/>
+</segment>
+</net>
+<net name="N$22" class="0">
+<segment>
+<pinref part="U$2" gate="G$1" pin="1"/>
+<pinref part="U$2" gate="G$1" pin="2"/>
+</segment>
+</net>
+<net name="N$23" class="0">
+<segment>
+<pinref part="U$2" gate="G$1" pin="3"/>
+<pinref part="U$2" gate="G$1" pin="4"/>
+</segment>
+</net>

Commit message: Update smiley
Parts:
- removed DB4: LED, florian:LED
- removed RB4: 1k, resistor:R-EU_R0402
- added RD8: 10k, resistor:R-EU_R0402
- added RD9: 1k, resistor:R-EU_R0402
Connections:
- new net N$45: IC1.PD3(INT1), RD8.2
- net +5V: now also RD9.1
- net GND: now also RD8.1; no longer DB4.C
- net MISO: no longer IC1.PB4(MISO), RB4.1
- net MOSI: no longer IC1.PB3(MOSI/OC2), RB3.1
- net N$11: now also IC1.PB5(SCK), RB5.1; no longer IC1.PD3(INT1), RD3.1
- net N$13: now also IC1.PB4(MISO), RB3.1; no longer IC1.PD5(T1), RD5.1
- net N$14: now also IC1.PB3(MOSI/OC2), RB2.1; no longer IC1.PD4(XCK/T0), RD4.1
- net N$15: now also IC1.PB2(SS/OC1B), RB1.1; no longer IC1.PD6(AIN0), RD6.1
- net N$16: now also IC1.PB1(OC1A), RB0.1; no longer IC1.PD7(AIN1), RD7.1
- net N$17: now also RD7.1; no longer RB0.1
- net N$18: now also IC1.PD7(AIN1), RD6.1; no longer IC1.PB1(OC1A), RB1.1
- net N$19: now also IC1.PD6(AIN0), RD5.1; no longer IC1.PB2(SS/OC1B), RB2.1
- net N$20: now also IC1.PD5(T1), RD4.1; no longer IC1.ADC6
- net N$43: now also IC1.PD4(XCK/T0), RD3.1; no longer DB4.A, RB4.2
- net SCK: no longer IC1.PB5(SCK), RB5.1
Other:
- moved on the sheet: DB0, DB1, DB2, DB3, DD3, DD4, DD5, DD6, DD7, RB0, RB1, RB2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

Commit message: Update library
Parts:
- removed JP1: (no value), SparkFun:M023.5MM
- added G1: CR2032H, florian:CR2032H
Connections:
- net +5V: now also G1.-; no longer JP1.1
- net GND: now also G1.+; no longer JP1.2
Changed lines of the file:
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@@
 <part name="GND4" library="supply1" deviceset="GND" device=""/>
 <part name="P+5" library="supply1" deviceset="+5V" device=""/>
-<part name="JP1" library="SparkFun" deviceset="M02" device="3.5MM"/>
 <part name="P+4" library="supply1" deviceset="+5V" device=""/>
 <part name="GND5" library="supply1" deviceset="GND" device=""/>
@@
 <part name="RD9" library="resistor" deviceset="R-EU_" device="R0402" value="1k"/>
 <part name="P+1" library="supply1" deviceset="+5V" device=""/>
+<part name="G1" library="florian" deviceset="CR2032H" device=""/>
 </parts>
 <sheets>
@@
 <instance part="GND4" gate="1" x="30.48" y="-7.62"/>
 <instance part="P+5" gate="1" x="38.1" y="2.54"/>
-<instance part="JP1" gate="G$1" x="0" y="20.32" rot="R180"/>
-<instance part="P+4" gate="1" x="-10.16" y="22.86"/>
-<instance part="GND5" gate="1" x="-10.16" y="15.24"/>
+<instance part="P+4" gate="1" x="-10.16" y="17.78" rot="R90"/>
+<instance part="GND5" gate="1" x="2.54" y="17.78" rot="R90"/>
 <instance part="P+6" gate="1" x="20.32" y="60.96"/>
 <instance part="GND6" gate="1" x="10.16" y="60.96"/>
@@
 <instance part="RD9" gate="G$1" x="139.7" y="25.4" rot="R90"/>
 <instance part="P+1" gate="1" x="139.7" y="15.24" rot="R180"/>
+<instance part="G1" gate="1" x="-2.54" y="17.78"/>
 </instances>
 <busses>
@@
 <wire x1="101.6" y1="33.02" x2="106.68" y2="33.02" width="0.1524" layer="91"/>
 <junction x="101.6" y="33.02"/>
+<junction x="106.68" y="33.02"/>
 </segment>
 </net>
@@
 <wire x1="101.6" y1="30.48" x2="106.68" y2="30.48" width="0.1524" layer="91"/>
 <junction x="101.6" y="30.48"/>
+<junction x="106.68" y="30.48"/>
 </segment>
 </net>
@@
 <pinref part="C2" gate="G$1" pin="2"/>
 <junction x="7.62" y="38.1"/>
+<junction x="35.56" y="35.56"/>
+<junction x="35.56" y="38.1"/>
 </segment>
 <segment>
@@
 </segment>
 <segment>
-<pinref part="JP1" gate="G$1" pin="2"/>
-<pinref part="GND5" gate="1" pin="GND"/>
-<wire x1="-7.62" y1="17.78" x2="-10.16" y2="17.78" width="0.1524" layer="91"/>
-</segment>
-<segment>
 <pinref part="IC1" gate="G$1" pin="GND"/>
 <pinref part="GND6" gate="1" pin="GND"/>
 <wire x1="35.56" y1="63.5" x2="10.16" y2="63.5" width="0.1524" layer="91"/>
+<junction x="10.16" y="63.5"/>
 </segment>
 <segment>
@@
 <wire x1="124.46" y1="22.86" x2="124.46" y2="27.94" width="0.1524" layer="91"/>
 </segment>
+<segment>
+<pinref part="G1" gate="1" pin="+"/>
+<pinref part="GND5" gate="1" pin="GND"/>
+<junction x="0" y="17.78"/>
+</segment>
 </net>
 <net name="N$1" class="0">
@@
 <pinref part="RB6" gate="G$1" pin="1"/>
 <wire x1="35.56" y1="50.8" x2="30.48" y2="50.8" width="0.1524" layer="91"/>
+<junction x="30.48" y="50.8"/>
+<junction x="35.56" y="50.8"/>
 </segment>
 </net>
@@
 <pinref part="C2" gate="G$1" pin="1"/>
 <wire x1="7.62" y1="30.48" x2="22.86" y2="30.48" width="0.1524" layer="91"/>
+<junction x="35.56" y="33.02"/>
+<junction x="35.56" y="30.48"/>
 </segment>
 <segment>
@@
 <pinref part="P+2" gate="1" pin="+5V"/>
 <wire x1="20.32" y1="68.58" x2="22.86" y2="68.58" width="0.1524" layer="91"/>
+<junction x="20.32" y="68.58"/>
+<junction x="22.86" y="68.58"/>
 </segment>
 <segment>
@@
 <pinref part="P+5" gate="1" pin="+5V"/>
 <wire x1="25.4" y1="0" x2="38.1" y2="0" width="0.1524" layer="91"/>
-</segment>
-<segment>
-<pinref part="P+4" gate="1" pin="+5V"/>
-<pinref part="JP1" gate="G$1" pin="1"/>
-<wire x1="-10.16" y1="20.32" x2="-7.62" y2="20.32" width="0.1524" layer="91"/>
 </segment>
 <segment>
@@
 <junction x="20.32" y="58.42"/>
 <junction x="22.86" y="58.42"/>
+<junction x="25.4" y="60.96"/>
+<junction x="35.56" y="58.42"/>
 </segment>
 <segment>
@@
 <pinref part="P+1" gate="1" pin="+5V"/>
 <wire x1="139.7" y1="20.32" x2="139.7" y2="17.78" width="0.1524" layer="91"/>
+</segment>
+<segment>
+<pinref part="G1" gate="1" pin="-"/>
+<pinref part="P+4" gate="1" pin="+5V"/>
+<junction x="-7.62" y="17.78"/>
 </segment>
 </net>
@@
 <pinref part="RB7" gate="G$1" pin="2"/>
 <wire x1="30.48" y1="45.72" x2="35.56" y2="45.72" width="0.1524" layer="91"/>
+<junction x="35.56" y="45.72"/>
+<junction x="30.48" y="45.72"/>
 </segment>
 </net>
@@
 <pinref part="R1" gate="G$1" pin="1"/>
 <wire x1="33.02" y1="68.58" x2="35.56" y2="68.58" width="0.1524" layer="91"/>
+<junction x="33.02" y="68.58"/>
+<junction x="35.56" y="68.58"/>
 </segment>
 <segment>
@@
 <pinref part="IC1" gate="G$1" pin="AREF"/>
 <wire x1="33.02" y1="60.96" x2="35.56" y2="60.96" width="0.1524" layer="91"/>
+<junction x="33.02" y="60.96"/>
+<junction x="35.56" y="60.96"/>
 </segment>
 </net>
@@
 <pinref part="RB5" gate="G$1" pin="1"/>
 <wire x1="83.82" y1="10.16" x2="91.44" y2="10.16" width="0.1524" layer="91"/>
+<junction x="83.82" y="10.16"/>
+<junction x="91.44" y="10.16"/>
 </segment>
 </net>
@@
 <pinref part="IC1" gate="G$1" pin="PB4(MISO)"/>
 <wire x1="91.44" y1="12.7" x2="83.82" y2="12.7" width="0.1524" layer="91"/>
+<junction x="83.82" y="12.7"/>
+<junction x="91.44" y="12.7"/>
 </segment>
 </net>
@@
 <pinref part="RB2" gate="G$1" pin="1"/>
 <wire x1="83.82" y1="15.24" x2="91.44" y2="15.24" width="0.1524" layer="91"/>
+<junction x="83.82" y="15.24"/>
+<junction x="91.44" y="15.24"/>
 </segment>
 </net>
@@
 <pinref part="IC1" gate="G$1" pin="PB2(SS/OC1B)"/>
 <wire x1="91.44" y1="17.78" x2="83.82" y2="17.78" width="0.1524" layer="91"/>
+<junction x="83.82" y="17.78"/>
+<junction x="91.44" y="17.78"/>
 </segment>
 </net>
@@
 <pinref part="RB0" gate="G$1" pin="1"/>
 <wire x1="83.82" y1="20.32" x2="91.44" y2="20.32" width="0.1524" layer="91"/>
+<junction x="83.82" y="20.32"/>
+<junction x="91.44" y="20.32"/>
 </segment>
 </net>
@@
 <pinref part="IC1" gate="G$1" pin="PB0(ICP)"/>
 <wire x1="91.44" y1="22.86" x2="83.82" y2="22.86" width="0.1524" layer="91"/>
+<junction x="83.82" y="22.86"/>
+<junction x="91.44" y="22.86"/>
 </segment>
 </net>
@@
 <pinref part="RD6" gate="G$1" pin="1"/>
 <wire x1="83.82" y1="27.94" x2="91.44" y2="27.94" width="0.1524" layer="91"/>
+<junction x="83.82" y="27.94"/>
+<junction x="91.44" y="27.94"/>
 </segment>
 </net>
@@
 <pinref part="IC1" gate="G$1" pin="PD6(AIN0)"/>
 <wire x1="91.44" y1="30.48" x2="83.82" y2="30.48" width="0.1524" layer="91"/>
+<junction x="83.82" y="30.48"/>
+<junction x="91.44" y="30.48"/>
 </segment>
 </net>
@@
 <pinref part="RD4" gate="G$1" pin="1"/>
 <wire x1="83.82" y1="33.02" x2="91.44" y2="33.02" width="0.1524" layer="91"/>
+<junction x="83.82" y="33.02"/>
+<junction x="91.44" y="33.02"/>
 </segment>
 </net>
@@
 <pinref part="IC1" gate="G$1" pin="PD4(XCK/T0)"/>
 <wire x1="91.44" y1="35.56" x2="83.82" y2="35.56" width="0.1524" layer="91"/>
+<junction x="83.82" y="35.56"/>
+<junction x="91.44" y="35.56"/>
 </segment>
 </net>
@@
 <wire x1="124.46" y1="38.1" x2="129.54" y2="38.1" width="0.1524" layer="91"/>
 <junction x="124.46" y="38.1"/>
-</segment>
-</net>
+<junction x="83.82" y="38.1"/>
+<junction x="129.54" y="38.1"/>
+</segment>
+</net>
